Commit message: add meshes
stl and re path to new pkg

File: src/morodim_description/urdf/morodim.urdf.xacro (robot description, xacro)
@@ -30,10 +30,10 @@
     <visual>
       <geometry>
-        <mesh filename="file:///$(find dummy_description)/meshes/link_0.stl"/>
-      </geometry>
-    </visual>
-    <collision>
-      <geometry>
-        <mesh filename="file:///$(find dummy_description)/meshes/link_0.stl"/>
+        <mesh filename="file:///$(find morodim_description)/meshes/link_0.stl"/>
+      </geometry>
+    </visual>
+    <collision>
+      <geometry>
+        <mesh filename="file:///$(find morodim_description)/meshes/link_0.stl"/>
       </geometry>
     </collision>
@@ -51,10 +51,10 @@
     <visual>
       <geometry>
-        <mesh filename="file:///$(find dummy_description)/meshes/link_1.stl"/>
-      </geometry>
-    </visual>
-    <collision>
-      <geometry>
-        <mesh filename="file:///$(find dummy_description)/meshes/link_1.stl"/>
+        <mesh filename="file:///$(find morodim_description)/meshes/link_1.stl"/>
+      </geometry>
+    </visual>
+    <collision>
+      <geometry>
+        <mesh filename="file:///$(find morodim_description)/meshes/link_1.stl"/>
       </geometry>
     </collision>
@@ -78,11 +78,11 @@
       <origin xyz="0.0 0.0 0.0" rpy="0 0 ${-3.14/2}"/>
       <geometry>
-        <mesh filename="file:///$(find dummy_description)/meshes/link_2.stl"/>
-      </geometry>
-    </visual>
-    <collision>
-      <origin xyz="0.0 0.0 0.0" rpy="0 0 ${-3.14/2}"/>
-      <geometry>
-        <mesh filename="file:///$(find dummy_description)/meshes/link_2.stl"/>
+        <mesh filename="file:///$(find morodim_description)/meshes/link_2.stl"/>
+      </geometry>
+    </visual>
+    <collision>
+      <origin xyz="0.0 0.0 0.0" rpy="0 0 ${-3.14/2}"/>
+      <geometry>
+        <mesh filename="file:///$(find morodim_description)/meshes/link_2.stl"/>
       </geometry>
     </collision>
@@ -106,11 +106,11 @@
       <origin xyz="0.0 0.0 0.0" rpy="0 0 ${-3.14/2}"/>
       <geometry>
-        <mesh filename="file:///$(find dummy_description)/meshes/link_3.stl"/>
-      </geometry>
-    </visual>
-    <collision>
-      <origin xyz="0.0 0.0 0.0" rpy="0 0 ${-3.14/2}"/>
-      <geometry>
-        <mesh filename="file:///$(find dummy_description)/meshes/link_3.stl"/>
+        <mesh filename="file:///$(find morodim_description)/meshes/link_3.stl"/>
+      </geometry>
+    </visual>
+    <collision>
+      <origin xyz="0.0 0.0 0.0" rpy="0 0 ${-3.14/2}"/>
+      <geometry>
+        <mesh filename="file:///$(find morodim_description)/meshes/link_3.stl"/>
       </geometry>
     </collision>
@@ -134,11 +134,11 @@
       <origin xyz="0.0 0.0 0.0" rpy="0 0 0"/>
       <geometry>
-        <mesh filename="file:///$(find dummy_description)/meshes/end_effector.stl"/>
-      </geometry>
-    </visual>
-    <collision>
-      <origin xyz="0.0 0.0 0.0" rpy="0 0 ${-3.14/2}"/>
-      <geometry>
-        <mesh filename="file:///$(find dummy_description)/meshes/end_effector.stl"/>
+        <mesh filename="file:///$(find morodim_description)/meshes/end_effector.stl"/>
+      </geometry>
+    </visual>
+    <collision>
+      <origin xyz="0.0 0.0 0.0" rpy="0 0 ${-3.14/2}"/>
+      <geometry>
+        <mesh filename="file:///$(find morodim_description)/meshes/end_effector.stl"/>
       </geometry>
     </collision>
